File: KiCAD_Ebike_Controller/LCD.sch (KiCad schematic (older format))
At the start: 9 parts

Commit message: schem done
Parts:
- added Q? (x2): BCV62, Package_TO_SOT_SMD:SOT-143, symbol Transistor_BJT:BCV62
- added R? (x2): R_Small, symbol Device:R_Small
Connections:
- wire segments 69 -> 85
Changed lines of the file:
@@
 Connection ~ 4850 4650
 Entry Wire Line
-	3350 3350 3450 3450
+	2100 3350 2200 3450
 Entry Wire Line
-	3350 3250 3450 3350
+	2100 3250 2200 3350
 Wire Bus Line
-	3350 3350 3350 3250
+	2100 3350 2100 3250
 Wire Bus Line
-	3350 3250 2350 3250
-Wire Wire Line
-	3450 3350 4350 3350
+	2100 3250 1100 3250
+Wire Wire Line
+	2200 3350 2800 3350
 Wire Wire Line
 	4350 3450 3450 3450
@@
 Text Notes 3350 3800 0    50   ~ 0
 I2C ADDR = 0x20
-Text HLabel 2350 3250 0    50   Input ~ 0
+Text HLabel 1100 3250 0    50   Input ~ 0
 LCD_I2C
-Text Label 2650 3250 0    50   ~ 0
+Text Label 1400 3250 0    50   ~ 0
 LCD_I2C_[1..2]
 Text Label 3750 3350 0    50   ~ 0
@@
 Text Notes 3100 1400 0    50   ~ 0
 Decoupling caps place close to ICs
+$Comp
+L Transistor_BJT:BCV62 Q?
+U 1 1 5FA332E6
+P 2600 2500
+F 0 "Q?" H 2050 2550 50  0000 L CNN
+F 1 "BCV62" H 2050 2450 50  0000 L CNN
+F 2 "Package_TO_SOT_SMD:SOT-143" H 2600 2500 50  0001 C CIN
+F 3 "https://assets.nexperia.com/documents/data-sheet/BCV62.pdf" H 2500 2500 50  0001 L CNN
+	1    2600 2500
+	1    0    0    -1
+$EndComp
+$Comp
+L Transistor_BJT:BCV62 Q?
+U 1 1 5FA33AEC
+P 3250 2500
+F 0 "Q?" H 3538 2546 50  0000 L CNN
+F 1 "BCV62" H 3538 2455 50  0000 L CNN
+F 2 "Package_TO_SOT_SMD:SOT-143" H 3250 2500 50  0001 C CIN
+F 3 "https://assets.nexperia.com/documents/data-sheet/BCV62.pdf" H 3150 2500 50  0001 L CNN
+	1    3250 2500
+	1    0    0    -1
+$EndComp
+$Comp
+L Device:R_Small R?
+U 1 1 5FA49804
+P 2400 2900
+F 0 "R?" H 2459 2946 50  0000 L CNN
+F 1 "R_Small" H 2459 2855 50  0000 L CNN
+F 2 "" H 2400 2900 50  0001 C CNN
+F 3 "~" H 2400 2900 50  0001 C CNN
+	1    2400 2900
+	1    0    0    -1
+$EndComp
+$Comp
+L Device:R_Small R?
+U 1 1 5FA49B10
+P 3050 2900
+F 0 "R?" H 3109 2946 50  0000 L CNN
+F 1 "R_Small" H 3109 2855 50  0000 L CNN
+F 2 "" H 3050 2900 50  0001 C CNN
+F 3 "~" H 3050 2900 50  0001 C CNN
+	1    3050 2900
+	1    0    0    -1
+$EndComp
+Wire Wire Line
+	2800 2700 2800 3350
+Connection ~ 2800 3350
+Wire Wire Line
+	2800 3350 4350 3350
+Wire Wire Line
+	3450 2700 3450 3450
+Connection ~ 3450 3450
+Wire Wire Line
+	3450 3450 2200 3450
+$Comp
+L power:GND #PWR?
+U 1 1 5FA4F5F7
+P 2400 3100
+F 0 "#PWR?" H 2400 2850 50  0001 C CNN
+F 1 "GND" H 2405 2927 50  0000 C CNN
+F 2 "" H 2400 3100 50  0001 C CNN
+F 3 "" H 2400 3100 50  0001 C CNN
+	1    2400 3100
+	1    0    0    -1
+$EndComp
+$Comp
+L power:GND #PWR?
+U 1 1 5FA5155C
+P 3050 3100
+F 0 "#PWR?" H 3050 2850 50  0001 C CNN
+F 1 "GND" H 3055 2927 50  0000 C CNN
+F 2 "" H 3050 3100 50  0001 C CNN
+F 3 "" H 3050 3100 50  0001 C CNN
+	1    3050 3100
+	1    0    0    -1
+$EndComp
+Wire Wire Line
+	3050 2700 3050 2800
+Wire Wire Line
+	2400 2700 2400 2800
+Wire Wire Line
+	2400 3000 2400 3100
+Wire Wire Line
+	3050 3000 3050 3100
+Wire Wire Line
+	2400 2300 2400 2150
+Wire Wire Line
+	2400 2150 2800 2150
+Wire Wire Line
+	3450 2150 3450 2300
+Wire Wire Line
+	3050 2300 3050 2150
+Connection ~ 3050 2150
+Wire Wire Line
+	3050 2150 3450 2150
+Wire Wire Line
+	2800 2300 2800 2150
+Connection ~ 2800 2150
+Wire Wire Line
+	2800 2150 3050 2150
+Wire Wire Line
+	3450 2150 3750 2150
+Connection ~ 3450 2150
+Text Label 3750 2150 2    50   ~ 0
++3.3v
 $EndSCHEMATC

Commit message: adding footprints
Parts:
- C24, C25: renamed from C?; footprint (none) -> Capacitor_SMD:C_0805_2012Metric_Pad1.15x1.40mm_HandSolder
- gave numbers to parts that had none: 11
Changed lines of the file:
@@
 $Descr A4 11693 8268
 encoding utf-8
-Sheet 6 7
+Sheet 5 7
 Title ""
 Date ""
@@
 $EndDescr
 $Comp
-L Interface_Expansion:PCF8574 U?
+L Interface_Expansion:PCF8574 U3
 U 1 1 5FB7F21B
 P 4850 3750
-F 0 "U?" H 4850 4631 50  0000 C CNN
+F 0 "U3" H 4850 4631 50  0000 C CNN
 F 1 "PCF8574" H 4850 4540 50  0000 C CNN
 F 2 "" H 4850 3750 50  0001 C CNN
@@
 Connection ~ 6700 4900
 $Comp
-L power:GND #PWR?
+L power:GND #PWR0123
 U 1 1 5FB8819C
 P 6700 5100
-F 0 "#PWR?" H 6700 4850 50  0001 C CNN
+F 0 "#PWR0123" H 6700 4850 50  0001 C CNN
 F 1 "GND" H 6705 4927 50  0000 C CNN
 F 2 "" H 6700 5100 50  0001 C CNN
@@
 	2250 1650 2250 1500
 $Comp
-L Device:C_Small C?
+L Device:C_Small C24
 U 1 1 5FB9BA0E
 P 2250 1400
-F 0 "C?" H 2342 1446 50  0000 L CNN
+F 0 "C24" H 2342 1446 50  0000 L CNN
 F 1 "100n" H 2342 1355 50  0000 L CNN
-F 2 "" H 2250 1400 50  0001 C CNN
+F 2 "Capacitor_SMD:C_0805_2012Metric_Pad1.15x1.40mm_HandSolder" H 2250 1400 50  0001 C CNN
 F 3 "~" H 2250 1400 50  0001 C CNN
 	1    2250 1400
@@
 Connection ~ 2250 1650
 $Comp
-L power:GND #PWR?
+L power:GND #PWR0124
 U 1 1 5FB8C650
 P 4850 4850
-F 0 "#PWR?" H 4850 4600 50  0001 C CNN
+F 0 "#PWR0124" H 4850 4600 50  0001 C CNN
 F 1 "GND" H 4855 4677 50  0000 C CNN
 F 2 "" H 4850 4850 50  0001 C CNN
@@
 $EndComp
 $Comp
-L power:GND #PWR?
+L power:GND #PWR0125
 U 1 1 5FB9EEFA
 P 3000 1800
-F 0 "#PWR?" H 3000 1550 50  0001 C CNN
+F 0 "#PWR0125" H 3000 1550 50  0001 C CNN
 F 1 "GND" H 3005 1627 50  0000 C CNN
 F 2 "" H 3000 1800 50  0001 C CNN
@@
 $EndComp
 $Comp
-L Device:R_Small R?
+L Device:R_Small R32
 U 1 1 5F9C9800
 P 7500 3200
-F 0 "R?" H 7559 3246 50  0000 L CNN
+F 0 "R32" H 7559 3246 50  0000 L CNN
 F 1 "50k" H 7559 3155 50  0000 L CNN
 F 2 "" H 7500 3200 50  0001 C CNN
@@
 $EndComp
 $Comp
-L Device:R_Small R?
+L Device:R_Small R33
 U 1 1 5F9C9C39
 P 7500 3500
-F 0 "R?" H 7559 3546 50  0000 L CNN
+F 0 "R33" H 7559 3546 50  0000 L CNN
 F 1 "50k" H 7559 3455 50  0000 L CNN
 F 2 "" H 7500 3500 50  0001 C CNN
@@
 	6700 4850 6700 4750
 $Comp
-L Display_Character:HY1602E DS?
+L Display_Character:HY1602E DS1
 U 1 1 5F9D0095
 P 6700 3950
-F 0 "DS?" H 7150 3400 50  0000 C CNN
+F 0 "DS1" H 7150 3400 50  0000 C CNN
 F 1 "HY1602E" H 7250 3300 50  0000 C CNN
 F 2 "Display:HY1602E" H 6700 3050 50  0001 C CIN
@@
 	6100 3550 6300 3550
 $Comp
-L Transistor_BJT:2N2219 Q?
+L Transistor_BJT:2N2219 Q9
 U 1 1 5F9D5255
 P 8050 4450
-F 0 "Q?" H 8241 4496 50  0000 L CNN
+F 0 "Q9" H 8241 4496 50  0000 L CNN
 F 1 "2N2219" H 8241 4405 50  0000 L CNN
 F 2 "Package_TO_SOT_THT:TO-39-3" H 8250 4375 50  0001 L CIN
@@
 $EndComp
 $Comp
-L Device:R_Small R?
+L Device:R_Small R34
 U 1 1 5F9D7B2B
 P 7950 3250
-F 0 "R?" H 8009 3296 50  0000 L CNN
+F 0 "R34" H 8009 3296 50  0000 L CNN
 F 1 "220" H 8009 3205 50  0000 L CNN
 F 2 "" H 7950 3250 50  0001 C CNN
@@
 	5600 5450 8500 5450
 $Comp
-L Device:R_Small R?
+L Device:R_Small R35
 U 1 1 5F9DE56C
 P 8500 4650
-F 0 "R?" H 8559 4696 50  0000 L CNN
+F 0 "R35" H 8559 4696 50  0000 L CNN
 F 1 "10k" H 8559 4605 50  0000 L CNN
 F 2 "" H 8500 4650 50  0001 C CNN
@@
 	7950 3000 8600 3000
 $Comp
-L Device:C_Small C?
+L Device:C_Small C25
 U 1 1 5F9F30E4
 P 2650 1400
-F 0 "C?" H 2742 1446 50  0000 L CNN
+F 0 "C25" H 2742 1446 50  0000 L CNN
 F 1 "100n" H 2742 1355 50  0000 L CNN
-F 2 "" H 2650 1400 50  0001 C CNN
+F 2 "Capacitor_SMD:C_0805_2012Metric_Pad1.15x1.40mm_HandSolder" H 2650 1400 50  0001 C CNN
 F 3 "~" H 2650 1400 50  0001 C CNN
 	1    2650 1400
@@
 Decoupling caps place close to ICs
 $Comp
-L Transistor_BJT:BCV62 Q?
+L Transistor_BJT:BCV62 Q7
 U 1 1 5FA332E6
 P 2600 2500
-F 0 "Q?" H 2050 2550 50  0000 L CNN
+F 0 "Q7" H 2050 2550 50  0000 L CNN
 F 1 "BCV62" H 2050 2450 50  0000 L CNN
 F 2 "Package_TO_SOT_SMD:SOT-143" H 2600 2500 50  0001 C CIN
@@
 $EndComp
 $Comp
-L Transistor_BJT:BCV62 Q?
+L Transistor_BJT:BCV62 Q8
 U 1 1 5FA33AEC
 P 3250 2500
-F 0 "Q?" H 3538 2546 50  0000 L CNN
+F 0 "Q8" H 3538 2546 50  0000 L CNN
 F 1 "BCV62" H 3538 2455 50  0000 L CNN
 F 2 "Package_TO_SOT_SMD:SOT-143" H 3250 2500 50  0001 C CIN
@@
 $EndComp
 $Comp
-L Device:R_Small R?
+L Device:R_Small R30
 U 1 1 5FA49804
 P 2400 2900
-F 0 "R?" H 2459 2946 50  0000 L CNN
+F 0 "R30" H 2459 2946 50  0000 L CNN
 F 1 "R_Small" H 2459 2855 50  0000 L CNN
 F 2 "" H 2400 2900 50  0001 C CNN
@@
 $EndComp
 $Comp
-L Device:R_Small R?
+L Device:R_Small R31
 U 1 1 5FA49B10
 P 3050 2900
-F 0 "R?" H 3109 2946 50  0000 L CNN
+F 0 "R31" H 3109 2946 50  0000 L CNN
 F 1 "R_Small" H 3109 2855 50  0000 L CNN
 F 2 "" H 3050 2900 50  0001 C CNN
@@
 	3450 3450 2200 3450
 $Comp
-L power:GND #PWR?
+L power:GND #PWR0126
 U 1 1 5FA4F5F7
 P 2400 3100
-F 0 "#PWR?" H 2400 2850 50  0001 C CNN
+F 0 "#PWR0126" H 2400 2850 50  0001 C CNN
 F 1 "GND" H 2405 2927 50  0000 C CNN
 F 2 "" H 2400 3100 50  0001 C CNN
@@
 $EndComp
 $Comp
-L power:GND #PWR?
+L power:GND #PWR0127
 U 1 1 5FA5155C
 P 3050 3100
-F 0 "#PWR?" H 3050 2850 50  0001 C CNN
+F 0 "#PWR0127" H 3050 2850 50  0001 C CNN
 F 1 "GND" H 3055 2927 50  0000 C CNN
 F 2 "" H 3050 3100 50  0001 C CNN

Commit message: 50% of the way through the layout
Parts:
- removed Q9: 2N2219, Package_TO_SOT_THT:TO-39-3, symbol Transistor_BJT:2N2219
- added J10: I2C_SCL, Connector_PinHeader_2.54mm:PinHeader_1x01_P2.54mm_Vertical, symbol Connector:Conn_01x01_Female
- added J11: I2C_SDA, Connector_PinHeader_2.54mm:PinHeader_1x01_P2.54mm_Vertical, symbol Connector:Conn_01x01_Female
- added Q9: 2N7000, Package_TO_SOT_THT:TO-92_Inline, symbol Transistor_FET:2N7000
- added R20: 100k, Resistor_SMD:R_0805_2012Metric_Pad1.15x1.40mm_HandSolder, symbol Device:R_Small
- R30, R31: value R_Small -> 4k7; footprint (none) -> Resistor_SMD:R_0805_2012Metric_Pad1.15x1.40mm_HandSolder
- R32, R33, R34: footprint (none) -> Resistor_SMD:R_0805_2012Metric_Pad1.15x1.40mm_HandSolder
- R35: value 10k -> 20; footprint (none) -> Resistor_SMD:R_0805_2012Metric_Pad1.15x1.40mm_HandSolder
- U3: footprint (none) -> Package_SO:SOIC-18W_7.5x11.6mm_P1.27mm
Connections:
- net labels added: GNDD
- wire segments 85 -> 94
Other:
- note added: "approx. 1mA current pull up"
- moved on the sheet: R35
Changed lines of the file:
@@
 $Descr A4 11693 8268
 encoding utf-8
-Sheet 5 7
+Sheet 4 7
 Title ""
 Date ""
@@
 F 0 "U3" H 4850 4631 50  0000 C CNN
 F 1 "PCF8574" H 4850 4540 50  0000 C CNN
-F 2 "" H 4850 3750 50  0001 C CNN
+F 2 "Package_SO:SOIC-18W_7.5x11.6mm_P1.27mm" H 4850 3750 50  0001 C CNN
 F 3 "http://www.nxp.com/documents/data_sheet/PCF8574_PCF8574A.pdf" H 4850 3750 50  0001 C CNN
 	1    4850 3750
@@
 	6700 4900 6700 5100
 Connection ~ 6700 4900
-$Comp
-L power:GND #PWR0123
-U 1 1 5FB8819C
-P 6700 5100
-F 0 "#PWR0123" H 6700 4850 50  0001 C CNN
-F 1 "GND" H 6705 4927 50  0000 C CNN
-F 2 "" H 6700 5100 50  0001 C CNN
-F 3 "" H 6700 5100 50  0001 C CNN
-	1    6700 5100
-	1    0    0    -1
-$EndComp
 Wire Wire Line
 	6700 3150 6700 3000
@@
 	2200 3350 2800 3350
 Wire Wire Line
-	4350 3450 3450 3450
+	4350 3450 4250 3450
 Wire Wire Line
 	6700 3000 4850 3000
@@
 Text Label 1400 3250 0    50   ~ 0
 LCD_I2C_[1..2]
-Text Label 3750 3350 0    50   ~ 0
+Text Label 3700 3350 0    50   ~ 0
 LCD_I2C_1
-Text Label 3750 3450 0    50   ~ 0
+Text Label 3700 3450 0    50   ~ 0
 LCD_I2C_2
 Text HLabel 1950 1150 0    50   Input ~ 0
@@
 Wire Wire Line
 	2250 1650 2650 1650
-Wire Wire Line
-	3000 1650 3000 1800
 Connection ~ 2250 1650
-$Comp
-L power:GND #PWR0124
-U 1 1 5FB8C650
-P 4850 4850
-F 0 "#PWR0124" H 4850 4600 50  0001 C CNN
-F 1 "GND" H 4855 4677 50  0000 C CNN
-F 2 "" H 4850 4850 50  0001 C CNN
-F 3 "" H 4850 4850 50  0001 C CNN
-	1    4850 4850
-	1    0    0    -1
-$EndComp
-$Comp
-L power:GND #PWR0125
-U 1 1 5FB9EEFA
-P 3000 1800
-F 0 "#PWR0125" H 3000 1550 50  0001 C CNN
-F 1 "GND" H 3005 1627 50  0000 C CNN
-F 2 "" H 3000 1800 50  0001 C CNN
-F 3 "" H 3000 1800 50  0001 C CNN
-	1    3000 1800
-	1    0    0    -1
-$EndComp
 $Comp
 L Device:R_Small R32
@@
 F 0 "R32" H 7559 3246 50  0000 L CNN
 F 1 "50k" H 7559 3155 50  0000 L CNN
-F 2 "" H 7500 3200 50  0001 C CNN
+F 2 "Resistor_SMD:R_0805_2012Metric_Pad1.15x1.40mm_HandSolder" H 7500 3200 50  0001 C CNN
 F 3 "~" H 7500 3200 50  0001 C CNN
 	1    7500 3200
@@
 F 0 "R33" H 7559 3546 50  0000 L CNN
 F 1 "50k" H 7559 3455 50  0000 L CNN
-F 2 "" H 7500 3500 50  0001 C CNN
+F 2 "Resistor_SMD:R_0805_2012Metric_Pad1.15x1.40mm_HandSolder" H 7500 3500 50  0001 C CNN
 F 3 "~" H 7500 3500 50  0001 C CNN
 	1    7500 3500
@@
 	6100 3550 6300 3550
 $Comp
-L Transistor_BJT:2N2219 Q9
-U 1 1 5F9D5255
-P 8050 4450
-F 0 "Q9" H 8241 4496 50  0000 L CNN
-F 1 "2N2219" H 8241 4405 50  0000 L CNN
-F 2 "Package_TO_SOT_THT:TO-39-3" H 8250 4375 50  0001 L CIN
-F 3 "http://www.onsemi.com/pub_link/Collateral/2N2219-D.PDF" H 8050 4450 50  0001 L CNN
-	1    8050 4450
-	-1   0    0    -1
-$EndComp
-$Comp
 L Device:R_Small R34
 U 1 1 5F9D7B2B
@@
 F 0 "R34" H 8009 3296 50  0000 L CNN
 F 1 "220" H 8009 3205 50  0000 L CNN
-F 2 "" H 7950 3250 50  0001 C CNN
+F 2 "Resistor_SMD:R_0805_2012Metric_Pad1.15x1.40mm_HandSolder" H 7950 3250 50  0001 C CNN
 F 3 "~" H 7950 3250 50  0001 C CNN
 	1    7950 3250
@@
 	7950 3150 7950 3000
 Wire Wire Line
-	8250 4450 8500 4450
-Wire Wire Line
 	5350 3950 5600 3950
 Wire Wire Line
 	5600 3950 5600 5450
 Wire Wire Line
-	5600 5450 8500 5450
+	5600 5450 8650 5450
 $Comp
 L Device:R_Small R35
 U 1 1 5F9DE56C
-P 8500 4650
-F 0 "R35" H 8559 4696 50  0000 L CNN
-F 1 "10k" H 8559 4605 50  0000 L CNN
-F 2 "" H 8500 4650 50  0001 C CNN
-F 3 "~" H 8500 4650 50  0001 C CNN
-	1    8500 4650
-	1    0    0    -1
-$EndComp
-Wire Wire Line
-	8500 4750 8500 5450
-Wire Wire Line
-	8500 4550 8500 4450
+P 8650 4650
+F 0 "R35" H 8709 4696 50  0000 L CNN
+F 1 "20" H 8709 4605 50  0000 L CNN
+F 2 "Resistor_SMD:R_0805_2012Metric_Pad1.15x1.40mm_HandSolder" H 8650 4650 50  0001 C CNN
+F 3 "~" H 8650 4650 50  0001 C CNN
+	1    8650 4650
+	1    0    0    -1
+$EndComp
+Wire Wire Line
+	8650 4750 8650 5450
+Wire Wire Line
+	8650 4550 8650 4450
 Wire Wire Line
 	7950 3350 7950 3950
@@
 Wire Wire Line
 	2650 1500 2650 1650
-Connection ~ 2650 1650
-Wire Wire Line
-	2650 1650 3000 1650
 Wire Wire Line
 	2650 1300 2650 1150
@@
 P 2400 2900
 F 0 "R30" H 2459 2946 50  0000 L CNN
-F 1 "R_Small" H 2459 2855 50  0000 L CNN
-F 2 "" H 2400 2900 50  0001 C CNN
+F 1 "4k7" H 2459 2855 50  0000 L CNN
+F 2 "Resistor_SMD:R_0805_2012Metric_Pad1.15x1.40mm_HandSolder" H 2400 2900 50  0001 C CNN
 F 3 "~" H 2400 2900 50  0001 C CNN
 	1    2400 2900
@@
 P 3050 2900
 F 0 "R31" H 3109 2946 50  0000 L CNN
-F 1 "R_Small" H 3109 2855 50  0000 L CNN
-F 2 "" H 3050 2900 50  0001 C CNN
+F 1 "4k7" H 3109 2855 50  0000 L CNN
+F 2 "Resistor_SMD:R_0805_2012Metric_Pad1.15x1.40mm_HandSolder" H 3050 2900 50  0001 C CNN
 F 3 "~" H 3050 2900 50  0001 C CNN
 	1    3050 2900
@@
 Connection ~ 2800 3350
 Wire Wire Line
-	2800 3350 4350 3350
+	2800 3350 4150 3350
 Wire Wire Line
 	3450 2700 3450 3450
@@
 Wire Wire Line
 	3450 3450 2200 3450
-$Comp
-L power:GND #PWR0126
-U 1 1 5FA4F5F7
-P 2400 3100
-F 0 "#PWR0126" H 2400 2850 50  0001 C CNN
-F 1 "GND" H 2405 2927 50  0000 C CNN
-F 2 "" H 2400 3100 50  0001 C CNN
-F 3 "" H 2400 3100 50  0001 C CNN
-	1    2400 3100
-	1    0    0    -1
-$EndComp
-$Comp
-L power:GND #PWR0127
-U 1 1 5FA5155C
-P 3050 3100
-F 0 "#PWR0127" H 3050 2850 50  0001 C CNN
-F 1 "GND" H 3055 2927 50  0000 C CNN
-F 2 "" H 3050 3100 50  0001 C CNN
-F 3 "" H 3050 3100 50  0001 C CNN
-	1    3050 3100
-	1    0    0    -1
-$EndComp
 Wire Wire Line
 	3050 2700 3050 2800
 Wire Wire Line
 	2400 2700 2400 2800
-Wire Wire Line
-	2400 3000 2400 3100
-Wire Wire Line
-	3050 3000 3050 3100
 Wire Wire Line
 	2400 2300 2400 2150
@@
 Text Label 3750 2150 2    50   ~ 0
 +3.3v
+$Comp
+L Transistor_FET:2N7000 Q9
+U 1 1 5FD63460
+P 8050 4450
+F 0 "Q9" H 8256 4496 50  0000 L CNN
+F 1 "2N7000" H 8256 4405 50  0000 L CNN
+F 2 "Package_TO_SOT_THT:TO-92_Inline" H 8250 4375 50  0001 L CIN
+F 3 "https://www.fairchildsemi.com/datasheets/2N/2N7000.pdf" H 8050 4450 50  0001 L CNN
+	1    8050 4450
+	-1   0    0    -1
+$EndComp
+$Comp
+L Device:R_Small R20
+U 1 1 5FD697B5
+P 8350 4700
+F 0 "R20" H 8409 4746 50  0000 L CNN
+F 1 "100k" H 8409 4655 50  0000 L CNN
+F 2 "Resistor_SMD:R_0805_2012Metric_Pad1.15x1.40mm_HandSolder" H 8350 4700 50  0001 C CNN
+F 3 "~" H 8350 4700 50  0001 C CNN
+	1    8350 4700
+	1    0    0    -1
+$EndComp
+Wire Wire Line
+	8350 4800 8350 4850
+Wire Wire Line
+	8350 4850 7950 4850
+Connection ~ 7950 4850
+Wire Wire Line
+	8350 4600 8350 4450
+Wire Wire Line
+	8350 4450 8250 4450
+Wire Wire Line
+	8650 4450 8350 4450
+Connection ~ 8350 4450
+Text Notes 1250 2900 0    50   ~ 0
+approx. 1mA current pull up
+$Comp
+L Connector:Conn_01x01_Female J10
+U 1 1 5FE6B53B
+P 4500 2150
+F 0 "J10" H 4528 2176 50  0000 L CNN
+F 1 "I2C_SCL" H 4528 2085 50  0000 L CNN
+F 2 "Connector_PinHeader_2.54mm:PinHeader_1x01_P2.54mm_Vertical" H 4500 2150 50  0001 C CNN
+F 3 "~" H 4500 2150 50  0001 C CNN
+	1    4500 2150
+	1    0    0    -1
+$EndComp
+$Comp
+L Connector:Conn_01x01_Female J11
+U 1 1 5FE6DC65
+P 4500 2300
+F 0 "J11" H 4528 2326 50  0000 L CNN
+F 1 "I2C_SDA" H 4528 2235 50  0000 L CNN
+F 2 "Connector_PinHeader_2.54mm:PinHeader_1x01_P2.54mm_Vertical" H 4500 2300 50  0001 C CNN
+F 3 "~" H 4500 2300 50  0001 C CNN
+	1    4500 2300
+	1    0    0    -1
+$EndComp
+Wire Wire Line
+	4300 2150 4150 2150
+Connection ~ 4150 3350
+Wire Wire Line
+	4150 3350 4350 3350
+Wire Wire Line
+	4300 2300 4250 2300
+Connection ~ 4250 3450
+Wire Wire Line
+	4250 3450 3450 3450
+Wire Wire Line
+	4150 2150 4150 3350
+Wire Wire Line
+	4250 2300 4250 3450
+Wire Wire Line
+	3050 3000 3050 3100
+Wire Wire Line
+	2400 3000 2400 3100
+Connection ~ 2650 1650
+Wire Wire Line
+	2650 1650 3000 1650
+$Comp
+L power:GNDD #PWR0124
+U 1 1 5FE98192
+P 3000 1650
+F 0 "#PWR0124" H 3000 1400 50  0001 C CNN
+F 1 "GNDD" H 3004 1495 50  0000 C CNN
+F 2 "" H 3000 1650 50  0001 C CNN
+F 3 "" H 3000 1650 50  0001 C CNN
+	1    3000 1650
+	1    0    0    -1
+$EndComp
+$Comp
+L power:GNDD #PWR0125
+U 1 1 5FE98C99
+P 2400 3100
+F 0 "#PWR0125" H 2400 2850 50  0001 C CNN
+F 1 "GNDD" H 2404 2945 50  0000 C CNN
+F 2 "" H 2400 3100 50  0001 C CNN
+F 3 "" H 2400 3100 50  0001 C CNN
+	1    2400 3100
+	1    0    0    -1
+$EndComp
+$Comp
+L power:GNDD #PWR0126
+U 1 1 5FE990AA
+P 3050 3100
+F 0 "#PWR0126" H 3050 2850 50  0001 C CNN
+F 1 "GNDD" H 3054 2945 50  0000 C CNN
+F 2 "" H 3050 3100 50  0001 C CNN
+F 3 "" H 3050 3100 50  0001 C CNN
+	1    3050 3100
+	1    0    0    -1
+$EndComp
+$Comp
+L power:GNDD #PWR0127
+U 1 1 5FE99BE3
+P 4850 4850
+F 0 "#PWR0127" H 4850 4600 50  0001 C CNN
+F 1 "GNDD" H 4854 4695 50  0000 C CNN
+F 2 "" H 4850 4850 50  0001 C CNN
+F 3 "" H 4850 4850 50  0001 C CNN
+	1    4850 4850
+	1    0    0    -1
+$EndComp
+$Comp
+L power:GNDD #PWR0128
+U 1 1 5FE9AA17
+P 6700 5100
+F 0 "#PWR0128" H 6700 4850 50  0001 C CNN
+F 1 "GNDD" H 6704 4945 50  0000 C CNN
+F 2 "" H 6700 5100 50  0001 C CNN
+F 3 "" H 6700 5100 50  0001 C CNN
+	1    6700 5100
+	1    0    0    -1
+$EndComp
 $EndSCHEMATC
