File: KiCAD_Ebike_Controller/MCU.sch (KiCad schematic (older format))
At the start: 8 parts

Commit message: close to being done, need to add current pull ups on i2c
Parts:
- added C?: C_Small, symbol Device:C_Small
- added R? (x3): 100k, symbol Device:R_Small
Connections:
- net labels added: +3.3v, MODE_SW_PB7
- net labels removed: +3v3
- wire segments 66 -> 84
Other:
- note added: "Decoupling Cap (place as close to IC as possible)"
- moved on the sheet: SW?
Changed lines of the file:
@@
 	5600 2700 5700 2700
 Wire Wire Line
-	5600 2700 5600 2550
-Text HLabel 5600 2550 1    50   Input ~ 0
-+3v3
-Wire Wire Line
 	5500 4700 5500 4800
 Wire Wire Line
 	5600 4800 5600 4700
-Text HLabel 5500 5100 3    50   Input ~ 0
+Text HLabel 1600 2300 0    50   Input ~ 0
 GND
 Text HLabel 7850 4500 2    50   Output ~ 0
@@
 	7850 4500 6100 4500
 Wire Wire Line
-	5000 3900 3300 3900
-Wire Wire Line
-	5000 4000 3300 4000
+	5000 4000 3000 4000
 Wire Wire Line
 	5000 4100 3300 4100
-Text HLabel 3300 3900 0    50   Input ~ 0
+Text HLabel 2550 3900 0    50   Input ~ 0
 HALL_A_PB0
-Text HLabel 3300 4000 0    50   Input ~ 0
+Text HLabel 2550 4000 0    50   Input ~ 0
 HALL_B_PB1
-Text HLabel 3300 4100 0    50   Input ~ 0
+Text HLabel 2550 4100 0    50   Input ~ 0
 HALL_C_PB2
-Text HLabel 3300 4200 0    50   Output ~ 0
+Text HLabel 2550 4200 0    50   Output ~ 0
 nBRAKE_PA13
-Text HLabel 3300 4300 0    50   Input ~ 0
+Text HLabel 2550 4300 0    50   Input ~ 0
 nFAULT_PA14
 Wire Wire Line
-	5000 4200 3300 4200
-Wire Wire Line
-	3300 4300 5000 4300
+	5000 4200 2550 4200
+Wire Wire Line
+	2550 4300 5000 4300
 Wire Wire Line
 	6100 4300 7850 4300
@@
 Wire Wire Line
 	5000 3000 4650 3000
-Text HLabel 3300 3000 0    50   Input ~ 0
+Text HLabel 2550 3000 0    50   Input ~ 0
 nRST
 $Comp
@@
 $EndComp
 Wire Wire Line
-	5500 4800 5500 5100
+	5500 4800 5500 4950
 Connection ~ 5500 4800
 Wire Wire Line
 	5500 4800 5600 4800
-$Comp
-L power:GND #PWR?
-U 1 1 5F9B226C
-P 3700 3650
-F 0 "#PWR?" H 3700 3400 50  0001 C CNN
-F 1 "GND" H 3705 3477 50  0000 C CNN
-F 2 "" H 3700 3650 50  0001 C CNN
-F 3 "" H 3700 3650 50  0001 C CNN
-	1    3700 3650
-	1    0    0    -1
-$EndComp
 Wire Wire Line
 	4400 3500 4300 3500
 Connection ~ 4400 3500
-$Comp
-L power:GND #PWR?
-U 1 1 5F9B499D
-P 5600 4900
-F 0 "#PWR?" H 5600 4650 50  0001 C CNN
-F 1 "GND" H 5605 4727 50  0000 C CNN
-F 2 "" H 5600 4900 50  0001 C CNN
-F 3 "" H 5600 4900 50  0001 C CNN
-	1    5600 4900
-	1    0    0    -1
-$EndComp
-Wire Wire Line
-	5600 4900 5600 4800
-Connection ~ 5600 4800
-Wire Wire Line
-	5000 4400 3300 4400
-Text HLabel 3300 4400 0    50   Input ~ 0
+Wire Wire Line
+	5000 4400 2550 4400
+Text HLabel 2550 4400 0    50   Input ~ 0
 BRAKE_SW_PB6
 Wire Wire Line
@@
 F 3 "~" H 3700 3450 50  0001 C CNN
 	1    3700 3250
-	0    -1   1    0
+	0    1    1    0
 $EndComp
 Wire Wire Line
@@
 Connection ~ 3700 3000
 Wire Wire Line
-	3700 3000 3300 3000
+	3700 3000 2550 3000
 Wire Wire Line
 	3700 3650 3700 3500
@@
 Wire Wire Line
 	4300 3200 5000 3200
+$Comp
+L Device:R_Small R?
+U 1 1 5FA92A6F
+P 2700 3700
+F 0 "R?" H 2759 3746 50  0000 L CNN
+F 1 "100k" H 2759 3655 50  0000 L CNN
+F 2 "" H 2700 3700 50  0001 C CNN
+F 3 "~" H 2700 3700 50  0001 C CNN
+	1    2700 3700
+	1    0    0    -1
+$EndComp
+$Comp
+L Device:R_Small R?
+U 1 1 5FA92C9E
+P 3000 3700
+F 0 "R?" H 3059 3746 50  0000 L CNN
+F 1 "100k" H 3059 3655 50  0000 L CNN
+F 2 "" H 3000 3700 50  0001 C CNN
+F 3 "~" H 3000 3700 50  0001 C CNN
+	1    3000 3700
+	1    0    0    -1
+$EndComp
+$Comp
+L Device:R_Small R?
+U 1 1 5FA92FB3
+P 3300 3700
+F 0 "R?" H 3359 3746 50  0000 L CNN
+F 1 "100k" H 3359 3655 50  0000 L CNN
+F 2 "" H 3300 3700 50  0001 C CNN
+F 3 "~" H 3300 3700 50  0001 C CNN
+	1    3300 3700
+	1    0    0    -1
+$EndComp
+Wire Wire Line
+	2550 3900 2700 3900
+Wire Wire Line
+	2700 3800 2700 3900
+Connection ~ 2700 3900
+Wire Wire Line
+	2700 3900 5000 3900
+Wire Wire Line
+	3000 3800 3000 4000
+Connection ~ 3000 4000
+Wire Wire Line
+	3000 4000 2550 4000
+Wire Wire Line
+	3300 3800 3300 4100
+Connection ~ 3300 4100
+Wire Wire Line
+	3300 4100 2550 4100
+Wire Wire Line
+	2700 3600 2700 3450
+Wire Wire Line
+	3000 3600 3000 3450
+Wire Wire Line
+	3300 3600 3300 3450
+Wire Wire Line
+	3300 3450 3000 3450
+Connection ~ 3000 3450
+Text HLabel 1600 1950 0    50   Input ~ 0
++3.3v
+$Comp
+L power:GND #PWR?
+U 1 1 5FABED44
+P 1950 2600
+F 0 "#PWR?" H 1950 2350 50  0001 C CNN
+F 1 "GND" H 1955 2427 50  0000 C CNN
+F 2 "" H 1950 2600 50  0001 C CNN
+F 3 "" H 1950 2600 50  0001 C CNN
+	1    1950 2600
+	1    0    0    -1
+$EndComp
+$Comp
+L power:GND #PWR?
+U 1 1 5FACF53C
+P 3700 3650
+F 0 "#PWR?" H 3700 3400 50  0001 C CNN
+F 1 "GND" H 3705 3477 50  0000 C CNN
+F 2 "" H 3700 3650 50  0001 C CNN
+F 3 "" H 3700 3650 50  0001 C CNN
+	1    3700 3650
+	1    0    0    -1
+$EndComp
+$Comp
+L power:GND #PWR?
+U 1 1 5FACFE3C
+P 5500 4950
+F 0 "#PWR?" H 5500 4700 50  0001 C CNN
+F 1 "GND" H 5505 4777 50  0000 C CNN
+F 2 "" H 5500 4950 50  0001 C CNN
+F 3 "" H 5500 4950 50  0001 C CNN
+	1    5500 4950
+	1    0    0    -1
+$EndComp
+Wire Wire Line
+	1600 2300 1950 2300
+Wire Wire Line
+	1950 2300 1950 2600
+Text Label 1950 1950 2    50   ~ 0
++3.3v
+$Comp
+L Device:C_Small C?
+U 1 1 5FB49C0D
+P 2100 2150
+F 0 "C?" H 2192 2196 50  0000 L CNN
+F 1 "C_Small" H 2192 2105 50  0000 L CNN
+F 2 "" H 2100 2150 50  0001 C CNN
+F 3 "~" H 2100 2150 50  0001 C CNN
+	1    2100 2150
+	1    0    0    -1
+$EndComp
+Text Label 6000 2700 2    50   ~ 0
++3.3v
+Wire Wire Line
+	2100 2250 2100 2300
+Wire Wire Line
+	2100 2300 1950 2300
+Connection ~ 1950 2300
+Wire Wire Line
+	2100 2050 2100 1950
+Wire Wire Line
+	1600 1950 2100 1950
+Text Notes 2150 2000 0    50   ~ 0
+Decoupling Cap (place as close to IC as possible)
+Connection ~ 5700 2700
+Wire Wire Line
+	5700 2700 6000 2700
+Text Label 2450 3450 0    50   ~ 0
++3.3v
+Wire Wire Line
+	2700 3450 3000 3450
+Wire Wire Line
+	2700 3450 2450 3450
+Connection ~ 2700 3450
+Wire Wire Line
+	5000 4500 2550 4500
 Wire Bus Line
 	7200 3900 7200 4100
 Wire Bus Line
 	7150 3500 7150 3800
+Text HLabel 2550 4500 0    50   Input ~ 0
+MODE_SW_PB7
 $EndSCHEMATC

Commit message: schem done
Parts:
- added C? (x3): 100n, symbol Device:C_Small
Connections:
- net labels added: HALL_C_PB3, MODE1_SW_PB7, MODE2_SW_PA3, SWCLK_PA14, SWDIO_PA13, nBRAKE_PB4, nFAULT_PB5
- net labels removed: AMB_LIGHT_PA3, HALL_C_PB2, MODE_SW_PB7, SWCLK, SWDIO, nBRAKE_PA13, nFAULT_PA14
- wire segments 84 -> 101
Other:
- note removed: "ADC_IN3"
Changed lines of the file:
@@
 Wire Wire Line
 	6100 3100 7850 3100
-Text Notes 6200 3200 0    50   ~ 0
-ADC_IN2
-Wire Wire Line
-	6100 3200 7850 3200
-Wire Wire Line
-	6100 3300 7850 3300
-Text Notes 6200 3300 0    50   ~ 0
-ADC_IN3
 Text Notes 6200 3600 0    50   ~ 0
 SPI1_MISO
@@
 Text HLabel 7850 3100 2    50   Input ~ 0
 I_BATT_MON_PA1
-Text HLabel 7850 3200 2    50   Input ~ 0
-THROTTLE_PA2
-Text HLabel 7850 3300 2    50   Input ~ 0
-AMB_LIGHT_PA3
+Text HLabel 7850 3800 2    50   Input ~ 0
+MODE2_SW_PA3
 Text HLabel 7850 3500 2    50   Input ~ 0
 SD_SPI
@@
 	7850 4500 6100 4500
 Wire Wire Line
-	5000 4000 3000 4000
-Wire Wire Line
-	5000 4100 3300 4100
+	5000 4100 3450 4100
 Text HLabel 2550 3900 0    50   Input ~ 0
 HALL_A_PB0
@@
 HALL_B_PB1
 Text HLabel 2550 4100 0    50   Input ~ 0
-HALL_C_PB2
+HALL_C_PB3
 Text HLabel 2550 4200 0    50   Output ~ 0
-nBRAKE_PA13
+nBRAKE_PB4
 Text HLabel 2550 4300 0    50   Input ~ 0
-nFAULT_PA14
+nFAULT_PB5
 Wire Wire Line
 	5000 4200 2550 4200
-Wire Wire Line
-	2550 4300 5000 4300
 Wire Wire Line
 	6100 4300 7850 4300
 Text HLabel 7850 4300 2    50   Output ~ 0
-SWDIO
+SWDIO_PA13
 Text HLabel 7850 4400 2    50   Output ~ 0
-SWCLK
+SWCLK_PA14
 Wire Wire Line
 	6100 4400 7850 4400
@@
 Connection ~ 2700 3900
 Wire Wire Line
-	2700 3900 5000 3900
+	2700 3900 2800 3900
 Wire Wire Line
 	3000 3800 3000 4000
@@
 Wire Wire Line
 	5000 4500 2550 4500
+Text HLabel 2550 4500 0    50   Input ~ 0
+MODE1_SW_PB7
+Text Notes 6200 3200 0    50   ~ 0
+ADC_IN2
+Text HLabel 7850 3200 2    50   Input ~ 0
+THROTTLE_PA2
+Wire Wire Line
+	6100 3200 7850 3200
+Wire Wire Line
+	7100 3800 7100 3850
+Wire Wire Line
+	7100 3850 7200 3850
+Wire Wire Line
+	7200 3850 7200 3800
+Wire Wire Line
+	6100 3800 7100 3800
+Wire Wire Line
+	7200 3800 7850 3800
+$Comp
+L Device:C_Small C?
+U 1 1 5FCC672D
+P 2800 4750
+F 0 "C?" H 2892 4796 50  0000 L CNN
+F 1 "100n" H 2892 4705 50  0000 L CNN
+F 2 "" H 2800 4750 50  0001 C CNN
+F 3 "~" H 2800 4750 50  0001 C CNN
+	1    2800 4750
+	1    0    0    -1
+$EndComp
+$Comp
+L Device:C_Small C?
+U 1 1 5FCC6C62
+P 3100 4750
+F 0 "C?" H 3192 4796 50  0000 L CNN
+F 1 "100n" H 3192 4705 50  0000 L CNN
+F 2 "" H 3100 4750 50  0001 C CNN
+F 3 "~" H 3100 4750 50  0001 C CNN
+	1    3100 4750
+	1    0    0    -1
+$EndComp
+$Comp
+L Device:C_Small C?
+U 1 1 5FCC70C3
+P 3450 4750
+F 0 "C?" H 3542 4796 50  0000 L CNN
+F 1 "100n" H 3542 4705 50  0000 L CNN
+F 2 "" H 3450 4750 50  0001 C CNN
+F 3 "~" H 3450 4750 50  0001 C CNN
+	1    3450 4750
+	1    0    0    -1
+$EndComp
+Wire Wire Line
+	2550 4300 5000 4300
+Wire Wire Line
+	2800 4650 2800 3900
+Connection ~ 2800 3900
+Wire Wire Line
+	2800 3900 5000 3900
+Wire Wire Line
+	3100 4650 3100 4000
+Wire Wire Line
+	3000 4000 3100 4000
+Connection ~ 3100 4000
+Wire Wire Line
+	3100 4000 5000 4000
+Wire Wire Line
+	3450 4100 3450 4650
+Connection ~ 3450 4100
+Wire Wire Line
+	3450 4100 3300 4100
+Wire Wire Line
+	2800 4850 2800 5000
+Wire Wire Line
+	2800 5000 3100 5000
+Wire Wire Line
+	3450 5000 3450 4850
+Wire Wire Line
+	3100 4850 3100 5000
+Connection ~ 3100 5000
+$Comp
+L power:GND #PWR?
+U 1 1 5FCE6083
+P 3200 5150
+F 0 "#PWR?" H 3200 4900 50  0001 C CNN
+F 1 "GND" H 3205 4977 50  0000 C CNN
+F 2 "" H 3200 5150 50  0001 C CNN
+F 3 "" H 3200 5150 50  0001 C CNN
+	1    3200 5150
+	1    0    0    -1
+$EndComp
+Wire Wire Line
+	3100 5000 3200 5000
+Wire Wire Line
+	3200 5150 3200 5000
+Connection ~ 3200 5000
+Wire Wire Line
+	3200 5000 3450 5000
 Wire Bus Line
 	7200 3900 7200 4100
 Wire Bus Line
 	7150 3500 7150 3800
-Text HLabel 2550 4500 0    50   Input ~ 0
-MODE_SW_PB7
 $EndSCHEMATC

Commit message: adding footprints
Parts:
- added C5: 10n, Capacitor_SMD:C_0603_1608Metric_Pad1.05x0.95mm_HandSolder, symbol Device:C_Small
- C10, C11, C6, C7, C8, C9: renamed from C?; footprint (none) -> Capacitor_SMD:C_0805_2012Metric
- C4: renamed from C?; value C_Small -> 10u; footprint (none) -> Capacitor_SMD:C_0805_2012Metric_Pad1.15x1.40mm_HandSolder
- gave numbers to parts that had none: 8
Connections:
- wire segments 101 -> 105
Changed lines of the file:
@@
 P 5600 3700
 AR Path="/5F8C2CD9" Ref="U?"  Part="1"
-AR Path="/5F8BD648/5F8C2CD9" Ref="U?"  Part="1"
-F 0 "U?" H 5900 2750 50  0000 C CNN
+AR Path="/5F8BD648/5F8C2CD9" Ref="U1"  Part="1"
+F 0 "U1" H 5900 2750 50  0000 C CNN
 F 1 "STM32F030K6Tx" H 6150 2650 50  0000 C CNN
 F 2 "Package_QFP:LQFP-32_7x7mm_P0.8mm" H 5100 2800 50  0001 R CNN
@@
 SPI1_NSS
 $Comp
-L Device:Crystal_GND2_Small Y?
+L Device:Crystal_GND2_Small Y1
 U 1 1 5F915CDC
 P 4800 3650
-F 0 "Y?" V 4800 3750 50  0000 L CNN
+F 0 "Y1" V 4800 3750 50  0000 L CNN
 F 1 "Crystal_GND2_Small" V 4800 2650 50  0001 L CNN
 F 2 "" H 4800 3650 50  0001 C CNN
@@
 $EndComp
 $Comp
-L Device:C_Small C?
+L Device:C_Small C11
 U 1 1 5F91903B
 P 4550 3800
-F 0 "C?" V 4500 3900 50  0000 C CNN
+F 0 "C11" V 4500 3900 50  0000 C CNN
 F 1 "10p" V 4600 3850 50  0000 L CNN
-F 2 "" H 4550 3800 50  0001 C CNN
+F 2 "Capacitor_SMD:C_0805_2012Metric" H 4550 3800 50  0001 C CNN
 F 3 "~" H 4550 3800 50  0001 C CNN
 	1    4550 3800
@@
 Connection ~ 4800 3800
 $Comp
-L Device:C_Small C?
+L Device:C_Small C10
 U 1 1 5F918C0D
 P 4550 3500
-F 0 "C?" V 4400 3600 50  0000 C CNN
+F 0 "C10" V 4400 3600 50  0000 C CNN
 F 1 "10p" V 4500 3550 50  0000 L CNN
-F 2 "" H 4550 3500 50  0001 C CNN
+F 2 "Capacitor_SMD:C_0805_2012Metric" H 4550 3500 50  0001 C CNN
 F 3 "~" H 4550 3500 50  0001 C CNN
 	1    4550 3500
@@
 nRST
 $Comp
-L Device:R_Small R?
+L Device:R_Small R20
 U 1 1 5F9AB9AE
 P 4650 2850
-F 0 "R?" H 4709 2896 50  0000 L CNN
+F 0 "R20" H 4709 2896 50  0000 L CNN
 F 1 "100k" H 4709 2805 50  0000 L CNN
 F 2 "" H 4650 2850 50  0001 C CNN
@@
 Connection ~ 5500 2700
 $Comp
-L Device:C_Small C?
+L Device:C_Small C9
 U 1 1 5F9AE892
 P 3950 3200
-F 0 "C?" H 4042 3246 50  0000 L CNN
+F 0 "C9" H 4042 3246 50  0000 L CNN
 F 1 "100n" H 4042 3155 50  0000 L CNN
-F 2 "" H 3950 3200 50  0001 C CNN
+F 2 "Capacitor_SMD:C_0805_2012Metric" H 3950 3200 50  0001 C CNN
 F 3 "~" H 3950 3200 50  0001 C CNN
 	1    3950 3200
@@
 	4650 3000 3950 3000
 $Comp
-L Switch:SW_Push SW?
+L Switch:SW_Push SW1
 U 1 1 5F9CEA7D
 P 3700 3250
-F 0 "SW?" V 3654 3202 50  0000 R CNN
+F 0 "SW1" V 3654 3202 50  0000 R CNN
 F 1 "SW_Push" V 3745 3202 50  0000 R CNN
 F 2 "" H 3700 3450 50  0001 C CNN
@@
 Connection ~ 3700 3500
 $Comp
-L Device:R_Small R?
+L Device:R_Small R19
 U 1 1 5F9F5270
 P 4300 3300
-F 0 "R?" H 4359 3346 50  0000 L CNN
+F 0 "R19" H 4359 3346 50  0000 L CNN
 F 1 "100k" H 4359 3255 50  0000 L CNN
 F 2 "" H 4300 3300 50  0001 C CNN
@@
 	4300 3200 5000 3200
 $Comp
-L Device:R_Small R?
+L Device:R_Small R16
 U 1 1 5FA92A6F
 P 2700 3700
-F 0 "R?" H 2759 3746 50  0000 L CNN
+F 0 "R16" H 2759 3746 50  0000 L CNN
 F 1 "100k" H 2759 3655 50  0000 L CNN
 F 2 "" H 2700 3700 50  0001 C CNN
@@
 $EndComp
 $Comp
-L Device:R_Small R?
+L Device:R_Small R17
 U 1 1 5FA92C9E
 P 3000 3700
-F 0 "R?" H 3059 3746 50  0000 L CNN
+F 0 "R17" H 3059 3746 50  0000 L CNN
 F 1 "100k" H 3059 3655 50  0000 L CNN
 F 2 "" H 3000 3700 50  0001 C CNN
@@
 $EndComp
 $Comp
-L Device:R_Small R?
+L Device:R_Small R18
 U 1 1 5FA92FB3
 P 3300 3700
-F 0 "R?" H 3359 3746 50  0000 L CNN
+F 0 "R18" H 3359 3746 50  0000 L CNN
 F 1 "100k" H 3359 3655 50  0000 L CNN
 F 2 "" H 3300 3700 50  0001 C CNN
@@
 +3.3v
 $Comp
-L power:GND #PWR?
+L power:GND #PWR0110
 U 1 1 5FABED44
 P 1950 2600
-F 0 "#PWR?" H 1950 2350 50  0001 C CNN
+F 0 "#PWR0110" H 1950 2350 50  0001 C CNN
 F 1 "GND" H 1955 2427 50  0000 C CNN
 F 2 "" H 1950 2600 50  0001 C CNN
@@
 $EndComp
 $Comp
-L power:GND #PWR?
+L power:GND #PWR0111
 U 1 1 5FACF53C
 P 3700 3650
-F 0 "#PWR?" H 3700 3400 50  0001 C CNN
+F 0 "#PWR0111" H 3700 3400 50  0001 C CNN
 F 1 "GND" H 3705 3477 50  0000 C CNN
 F 2 "" H 3700 3650 50  0001 C CNN
@@
 $EndComp
 $Comp
-L power:GND #PWR?
+L power:GND #PWR0112
 U 1 1 5FACFE3C
 P 5500 4950
-F 0 "#PWR?" H 5500 4700 50  0001 C CNN
+F 0 "#PWR0112" H 5500 4700 50  0001 C CNN
 F 1 "GND" H 5505 4777 50  0000 C CNN
 F 2 "" H 5500 4950 50  0001 C CNN
@@
 +3.3v
 $Comp
-L Device:C_Small C?
+L Device:C_Small C4
 U 1 1 5FB49C0D
 P 2100 2150
-F 0 "C?" H 2192 2196 50  0000 L CNN
-F 1 "C_Small" H 2192 2105 50  0000 L CNN
-F 2 "" H 2100 2150 50  0001 C CNN
+F 0 "C4" H 2192 2196 50  0000 L CNN
+F 1 "10u" H 2192 2105 50  0000 L CNN
+F 2 "Capacitor_SMD:C_0805_2012Metric_Pad1.15x1.40mm_HandSolder" H 2100 2150 50  0001 C CNN
 F 3 "~" H 2100 2150 50  0001 C CNN
 	1    2100 2150
@@
 Wire Wire Line
 	1600 1950 2100 1950
-Text Notes 2150 2000 0    50   ~ 0
+Text Notes 2250 1850 0    50   ~ 0
 Decoupling Cap (place as close to IC as possible)
 Connection ~ 5700 2700
@@
 	7200 3800 7850 3800
 $Comp
-L Device:C_Small C?
+L Device:C_Small C6
 U 1 1 5FCC672D
 P 2800 4750
-F 0 "C?" H 2892 4796 50  0000 L CNN
+F 0 "C6" H 2892 4796 50  0000 L CNN
 F 1 "100n" H 2892 4705 50  0000 L CNN
-F 2 "" H 2800 4750 50  0001 C CNN
+F 2 "Capacitor_SMD:C_0805_2012Metric" H 2800 4750 50  0001 C CNN
 F 3 "~" H 2800 4750 50  0001 C CNN
 	1    2800 4750
@@
 $EndComp
 $Comp
-L Device:C_Small C?
+L Device:C_Small C7
 U 1 1 5FCC6C62
 P 3100 4750
-F 0 "C?" H 3192 4796 50  0000 L CNN
+F 0 "C7" H 3192 4796 50  0000 L CNN
 F 1 "100n" H 3192 4705 50  0000 L CNN
-F 2 "" H 3100 4750 50  0001 C CNN
+F 2 "Capacitor_SMD:C_0805_2012Metric" H 3100 4750 50  0001 C CNN
 F 3 "~" H 3100 4750 50  0001 C CNN
 	1    3100 4750
@@
 $EndComp
 $Comp
-L Device:C_Small C?
+L Device:C_Small C8
 U 1 1 5FCC70C3
 P 3450 4750
-F 0 "C?" H 3542 4796 50  0000 L CNN
+F 0 "C8" H 3542 4796 50  0000 L CNN
 F 1 "100n" H 3542 4705 50  0000 L CNN
-F 2 "" H 3450 4750 50  0001 C CNN
+F 2 "Capacitor_SMD:C_0805_2012Metric" H 3450 4750 50  0001 C CNN
 F 3 "~" H 3450 4750 50  0001 C CNN
 	1    3450 4750
@@
 Connection ~ 3100 5000
 $Comp
-L power:GND #PWR?
+L power:GND #PWR0113
 U 1 1 5FCE6083
 P 3200 5150
-F 0 "#PWR?" H 3200 4900 50  0001 C CNN
+F 0 "#PWR0113" H 3200 4900 50  0001 C CNN
 F 1 "GND" H 3205 4977 50  0000 C CNN
 F 2 "" H 3200 5150 50  0001 C CNN
@@
 Wire Wire Line
 	3200 5000 3450 5000
+$Comp
+L Device:C_Small C5
+U 1 1 5FC996AA
+P 2450 2150
+F 0 "C5" H 2542 2196 50  0000 L CNN
+F 1 "10n" H 2542 2105 50  0000 L CNN
+F 2 "Capacitor_SMD:C_0603_1608Metric_Pad1.05x0.95mm_HandSolder" H 2450 2150 50  0001 C CNN
+F 3 "~" H 2450 2150 50  0001 C CNN
+	1    2450 2150
+	1    0    0    -1
+$EndComp
+Wire Wire Line
+	2450 2050 2450 1950
+Wire Wire Line
+	2450 1950 2100 1950
+Connection ~ 2100 1950
+Wire Wire Line
+	2450 2250 2450 2300
+Wire Wire Line
+	2450 2300 2100 2300
 Wire Bus Line
 	7200 3900 7200 4100
 Wire Bus Line
 	7150 3500 7150 3800
+Connection ~ 2100 2300
 $EndSCHEMATC
