File: KiCAD_Ebike_Controller/Triple_H_Bridge.sch (KiCad schematic (older format))
At the start: 24 parts

Commit message: adding footprints
Parts:
- gave numbers to parts that had none: 24
Connections:
- wire segments 84 -> 83
Changed lines of the file:
@@
 AR Path="/5FEC55C0" Ref="R?"  Part="1"
 AR Path="/5F8D3A83/5FEC55C0" Ref="R?"  Part="1"
-AR Path="/5FECEF22/5FEC55C0" Ref="R?"  Part="1"
-F 0 "R?" V 3543 2400 50  0000 C CNN
+AR Path="/5FECEF22/5FEC55C0" Ref="R4"  Part="1"
+F 0 "R4" V 3543 2400 50  0000 C CNN
 F 1 "20m" V 3634 2400 50  0000 C CNN
 F 2 "" V 3680 2400 50  0001 C CNN
@@
 P 4100 2400
 AR Path="/5F8D3A83/5FEC55C9" Ref="D?"  Part="1"
-AR Path="/5FECEF22/5FEC55C9" Ref="D?"  Part="1"
-F 0 "D?" H 4100 2616 50  0000 C CNN
+AR Path="/5FECEF22/5FEC55C9" Ref="D1"  Part="1"
+F 0 "D1" H 4100 2616 50  0000 C CNN
 F 1 "1N47xxA" H 4100 2525 50  0000 C CNN
 F 2 "Diode_THT:D_DO-41_SOD81_P10.16mm_Horizontal" H 4100 2225 50  0001 C CNN
@@
 AR Path="/5FEC55CF" Ref="R?"  Part="1"
 AR Path="/5F8D3A83/5FEC55CF" Ref="R?"  Part="1"
-AR Path="/5FECEF22/5FEC55CF" Ref="R?"  Part="1"
-F 0 "R?" V 3743 2600 50  0000 C CNN
+AR Path="/5FECEF22/5FEC55CF" Ref="R6"  Part="1"
+F 0 "R6" V 3743 2600 50  0000 C CNN
 F 1 "20m" V 3834 2600 50  0000 C CNN
 F 2 "" V 3880 2600 50  0001 C CNN
@@
 AR Path="/5FEC55D5" Ref="R?"  Part="1"
 AR Path="/5F8D3A83/5FEC55D5" Ref="R?"  Part="1"
-AR Path="/5FECEF22/5FEC55D5" Ref="R?"  Part="1"
-F 0 "R?" V 3543 3500 50  0000 C CNN
+AR Path="/5FECEF22/5FEC55D5" Ref="R5"  Part="1"
+F 0 "R5" V 3543 3500 50  0000 C CNN
 F 1 "20m" V 3634 3500 50  0000 C CNN
 F 2 "" V 3680 3500 50  0001 C CNN
@@
 P 4100 3500
 AR Path="/5F8D3A83/5FEC55DE" Ref="D?"  Part="1"
-AR Path="/5FECEF22/5FEC55DE" Ref="D?"  Part="1"
-F 0 "D?" H 4100 3716 50  0000 C CNN
+AR Path="/5FECEF22/5FEC55DE" Ref="D2"  Part="1"
+F 0 "D2" H 4100 3716 50  0000 C CNN
 F 1 "1N47xxA" H 4100 3625 50  0000 C CNN
 F 2 "Diode_THT:D_DO-41_SOD81_P10.16mm_Horizontal" H 4100 3325 50  0001 C CNN
@@
 AR Path="/5FEC55E5" Ref="R?"  Part="1"
 AR Path="/5F8D3A83/5FEC55E5" Ref="R?"  Part="1"
-AR Path="/5FECEF22/5FEC55E5" Ref="R?"  Part="1"
-F 0 "R?" V 3893 3700 50  0000 C CNN
+AR Path="/5FECEF22/5FEC55E5" Ref="R7"  Part="1"
+F 0 "R7" V 3893 3700 50  0000 C CNN
 F 1 "20m" V 3984 3700 50  0000 C CNN
 F 2 "" V 4030 3700 50  0001 C CNN
@@
 AR Path="/5FEC55F7" Ref="R?"  Part="1"
 AR Path="/5F8D3A83/5FEC55F7" Ref="R?"  Part="1"
-AR Path="/5FECEF22/5FEC55F7" Ref="R?"  Part="1"
-F 0 "R?" V 5593 2400 50  0000 C CNN
+AR Path="/5FECEF22/5FEC55F7" Ref="R9"  Part="1"
+F 0 "R9" V 5593 2400 50  0000 C CNN
 F 1 "20m" V 5684 2400 50  0000 C CNN
 F 2 "" V 5730 2400 50  0001 C CNN
@@
 P 6250 2400
 AR Path="/5F8D3A83/5FEC5600" Ref="D?"  Part="1"
-AR Path="/5FECEF22/5FEC5600" Ref="D?"  Part="1"
-F 0 "D?" H 6250 2616 50  0000 C CNN
+AR Path="/5FECEF22/5FEC5600" Ref="D4"  Part="1"
+F 0 "D4" H 6250 2616 50  0000 C CNN
 F 1 "1N47xxA" H 6250 2525 50  0000 C CNN
 F 2 "Diode_THT:D_DO-41_SOD81_P10.16mm_Horizontal" H 6250 2225 50  0001 C CNN
@@
 AR Path="/5FEC5606" Ref="R?"  Part="1"
 AR Path="/5F8D3A83/5FEC5606" Ref="R?"  Part="1"
-AR Path="/5FECEF22/5FEC5606" Ref="R?"  Part="1"
-F 0 "R?" V 5843 2600 50  0000 C CNN
+AR Path="/5FECEF22/5FEC5606" Ref="R11"  Part="1"
+F 0 "R11" V 5843 2600 50  0000 C CNN
 F 1 "20m" V 5934 2600 50  0000 C CNN
 F 2 "" V 5980 2600 50  0001 C CNN
@@
 AR Path="/5FEC560C" Ref="R?"  Part="1"
 AR Path="/5F8D3A83/5FEC560C" Ref="R?"  Part="1"
-AR Path="/5FECEF22/5FEC560C" Ref="R?"  Part="1"
-F 0 "R?" V 5543 3500 50  0000 C CNN
+AR Path="/5FECEF22/5FEC560C" Ref="R8"  Part="1"
+F 0 "R8" V 5543 3500 50  0000 C CNN
 F 1 "20m" V 5634 3500 50  0000 C CNN
 F 2 "" V 5680 3500 50  0001 C CNN
@@
 P 6200 3500
 AR Path="/5F8D3A83/5FEC5615" Ref="D?"  Part="1"
-AR Path="/5FECEF22/5FEC5615" Ref="D?"  Part="1"
-F 0 "D?" H 6200 3716 50  0000 C CNN
+AR Path="/5FECEF22/5FEC5615" Ref="D3"  Part="1"
+F 0 "D3" H 6200 3716 50  0000 C CNN
 F 1 "1N47xxA" H 6200 3625 50  0000 C CNN
 F 2 "Diode_THT:D_DO-41_SOD81_P10.16mm_Horizontal" H 6200 3325 50  0001 C CNN
@@
 AR Path="/5FEC561C" Ref="R?"  Part="1"
 AR Path="/5F8D3A83/5FEC561C" Ref="R?"  Part="1"
-AR Path="/5FECEF22/5FEC561C" Ref="R?"  Part="1"
-F 0 "R?" V 5793 3700 50  0000 C CNN
+AR Path="/5FECEF22/5FEC561C" Ref="R10"  Part="1"
+F 0 "R10" V 5793 3700 50  0000 C CNN
 F 1 "20m" V 5884 3700 50  0000 C CNN
 F 2 "" V 5930 3700 50  0001 C CNN
@@
 AR Path="/5FEC562C" Ref="R?"  Part="1"
 AR Path="/5F8D3A83/5FEC562C" Ref="R?"  Part="1"
-AR Path="/5FECEF22/5FEC562C" Ref="R?"  Part="1"
-F 0 "R?" V 7893 2400 50  0000 C CNN
+AR Path="/5FECEF22/5FEC562C" Ref="R13"  Part="1"
+F 0 "R13" V 7893 2400 50  0000 C CNN
 F 1 "20m" V 7984 2400 50  0000 C CNN
 F 2 "" V 8030 2400 50  0001 C CNN
@@
 P 8550 2400
 AR Path="/5F8D3A83/5FEC5635" Ref="D?"  Part="1"
-AR Path="/5FECEF22/5FEC5635" Ref="D?"  Part="1"
-F 0 "D?" H 8550 2616 50  0000 C CNN
+AR Path="/5FECEF22/5FEC5635" Ref="D6"  Part="1"
+F 0 "D6" H 8550 2616 50  0000 C CNN
 F 1 "1N47xxA" H 8550 2525 50  0000 C CNN
 F 2 "Diode_THT:D_DO-41_SOD81_P10.16mm_Horizontal" H 8550 2225 50  0001 C CNN
@@
 AR Path="/5FEC563B" Ref="R?"  Part="1"
 AR Path="/5F8D3A83/5FEC563B" Ref="R?"  Part="1"
-AR Path="/5FECEF22/5FEC563B" Ref="R?"  Part="1"
-F 0 "R?" V 8143 2600 50  0000 C CNN
+AR Path="/5FECEF22/5FEC563B" Ref="R15"  Part="1"
+F 0 "R15" V 8143 2600 50  0000 C CNN
 F 1 "20m" V 8234 2600 50  0000 C CNN
 F 2 "" V 8280 2600 50  0001 C CNN
@@
 AR Path="/5FEC5641" Ref="R?"  Part="1"
 AR Path="/5F8D3A83/5FEC5641" Ref="R?"  Part="1"
-AR Path="/5FECEF22/5FEC5641" Ref="R?"  Part="1"
-F 0 "R?" V 7843 3500 50  0000 C CNN
+AR Path="/5FECEF22/5FEC5641" Ref="R12"  Part="1"
+F 0 "R12" V 7843 3500 50  0000 C CNN
 F 1 "20m" V 7934 3500 50  0000 C CNN
 F 2 "" V 7980 3500 50  0001 C CNN
@@
 P 8500 3500
 AR Path="/5F8D3A83/5FEC564A" Ref="D?"  Part="1"
-AR Path="/5FECEF22/5FEC564A" Ref="D?"  Part="1"
-F 0 "D?" H 8500 3716 50  0000 C CNN
+AR Path="/5FECEF22/5FEC564A" Ref="D5"  Part="1"
+F 0 "D5" H 8500 3716 50  0000 C CNN
 F 1 "1N47xxA" H 8500 3625 50  0000 C CNN
 F 2 "Diode_THT:D_DO-41_SOD81_P10.16mm_Horizontal" H 8500 3325 50  0001 C CNN
@@
 AR Path="/5FEC5651" Ref="R?"  Part="1"
 AR Path="/5F8D3A83/5FEC5651" Ref="R?"  Part="1"
-AR Path="/5FECEF22/5FEC5651" Ref="R?"  Part="1"
-F 0 "R?" V 8093 3700 50  0000 C CNN
+AR Path="/5FECEF22/5FEC5651" Ref="R14"  Part="1"
+F 0 "R14" V 8093 3700 50  0000 C CNN
 F 1 "20m" V 8184 3700 50  0000 C CNN
 F 2 "" V 8230 3700 50  0001 C CNN
@@
 	4650 2750 4650 3000
 Wire Wire Line
-	10150 2850 6750 2850
+	10050 2850 6750 2850
 Wire Wire Line
 	6750 3000 6750 2850
@@
 P 4550 2400
 AR Path="/5F8D3A83/5FEC568A" Ref="Q?"  Part="1"
-AR Path="/5FECEF22/5FEC568A" Ref="Q?"  Part="1"
-F 0 "Q?" H 4756 2446 50  0000 L CNN
+AR Path="/5FECEF22/5FEC568A" Ref="Q1"  Part="1"
+F 0 "Q1" H 4756 2446 50  0000 L CNN
 F 1 "DMT10H010LK3" H 4400 2150 50  0000 L CNN
 F 2 "" H 4750 2500 50  0001 C CNN
@@
 P 4550 3500
 AR Path="/5F8D3A83/5FEC5691" Ref="Q?"  Part="1"
-AR Path="/5FECEF22/5FEC5691" Ref="Q?"  Part="1"
-F 0 "Q?" H 4756 3546 50  0000 L CNN
+AR Path="/5FECEF22/5FEC5691" Ref="Q2"  Part="1"
+F 0 "Q2" H 4756 3546 50  0000 L CNN
 F 1 "DMT10H010LK3" H 4400 3250 50  0000 L CNN
 F 2 "" H 4750 3600 50  0001 C CNN
@@
 P 6650 3500
 AR Path="/5F8D3A83/5FEC5699" Ref="Q?"  Part="1"
-AR Path="/5FECEF22/5FEC5699" Ref="Q?"  Part="1"
-F 0 "Q?" H 6856 3546 50  0000 L CNN
+AR Path="/5FECEF22/5FEC5699" Ref="Q4"  Part="1"
+F 0 "Q4" H 6856 3546 50  0000 L CNN
 F 1 "DMT10H010LK3" H 6500 3250 50  0000 L CNN
 F 2 "" H 6850 3600 50  0001 C CNN
@@
 P 8950 3500
 AR Path="/5F8D3A83/5FEC56A0" Ref="Q?"  Part="1"
-AR Path="/5FECEF22/5FEC56A0" Ref="Q?"  Part="1"
-F 0 "Q?" H 9156 3546 50  0000 L CNN
+AR Path="/5FECEF22/5FEC56A0" Ref="Q6"  Part="1"
+F 0 "Q6" H 9156 3546 50  0000 L CNN
 F 1 "DMT10H010LK3" H 8800 3250 50  0000 L CNN
 F 2 "" H 9150 3600 50  0001 C CNN
@@
 P 8950 2400
 AR Path="/5F8D3A83/5FEC56A7" Ref="Q?"  Part="1"
-AR Path="/5FECEF22/5FEC56A7" Ref="Q?"  Part="1"
-F 0 "Q?" H 9156 2446 50  0000 L CNN
+AR Path="/5FECEF22/5FEC56A7" Ref="Q5"  Part="1"
+F 0 "Q5" H 9156 2446 50  0000 L CNN
 F 1 "DMT10H010LK3" H 8800 2150 50  0000 L CNN
 F 2 "" H 9150 2500 50  0001 C CNN
@@
 P 6650 2400
 AR Path="/5F8D3A83/5FEC56AE" Ref="Q?"  Part="1"
-AR Path="/5FECEF22/5FEC56AE" Ref="Q?"  Part="1"
-F 0 "Q?" H 6856 2446 50  0000 L CNN
+AR Path="/5FECEF22/5FEC56AE" Ref="Q3"  Part="1"
+F 0 "Q3" H 6856 2446 50  0000 L CNN
 F 1 "DMT10H010LK3" H 6500 2150 50  0000 L CNN
 F 2 "" H 6850 2500 50  0001 C CNN
@@
 Wire Wire Line
 	6750 1400 6750 1900
-Wire Wire Line
-	6750 2850 6050 2850
 Wire Bus Line
 	1350 3800 3150 3800

Commit message: 50% of the way through the layout
Parts:
- removed D1, D2, D3, D4, D5, D6: 1N47xxA, Diode_THT:D_DO-41_SOD81_P10.16mm_Horizontal, symbol Diode:1N47xxA
- added D1, D2, D3, D4, D5, D6: SM4007, Diode_SMD:D_MELF, symbol Diode:SM4007
- Q1, Q2, Q3, Q4, Q5, Q6: footprint (none) -> Package_TO_SOT_SMD:TO-252-3_TabPin2
- R10, R11, R12, R13, R14, R15, R4, R5, R6, R7, R8, R9: value 20m -> 5; footprint (none) -> Resistor_SMD:R_0805_2012Metric_Pad1.15x1.40mm_HandSolder
Connections:
- net labels added: PA1, PA2, PA3, PA[1..3], PB1, PB2, PB3, PB[1..3], PC1, PC2, PC3, PC[1..3]
- net labels removed: PA_1, PA_2, PA_3, PA_[1..3], PB_1, PB_2, PB_3, PB_[1..3], PC_1, PC_2, PC_3, PC_[1..3], PHASE_A_FETs, PHASE_B_FETs, PHASE_C_FETs
- wire segments 83 -> 82
Other:
- moved on the sheet: R4

Commit message: Finished ready for fab
Parts:
- added RT1, RT2, RT3, RT4, RT5, RT6: R_Thermal, Resistor_SMD:R_1206_3216Metric_Pad1.42x1.75mm_HandSolder, symbol Device:R_Thermal
Connections:
- net +48V: now also RT1.1, RT3.1, RT5.1
- net PHASE_A: now also RT2.1
- net PHASE_B: now also RT4.1
- net PHASE_C: now also RT6.1
- new net GND: RT1.2, RT2.2, RT3.2, RT4.2, RT5.2, RT6.2
Other:
- moved on the sheet: D1, D2, D5, D6, Q1, Q2, Q5, Q6, R12, R13, R14, R15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
